File: bldc-hardware-master/design/BLDC_4.kicad_pcb (KiCad board)
At the start: 4 copper layers, 38.5 x 75 mm, 132 parts, among them J1 7466103, J2 7466103, J3 7466103, J4 7466103, J5 7466103, K1 SERVO, P1 HALL/Encoder, P101 CANBUS, P2 SWD, P3 PWR_COMM, P4 IN+, P5 IN-, P6 MOTOR1, P7 MOTOR2, P9 MOTOR3, Q1 IRFS7530, Q2 IRFS7530, Q3 IRFS7530, Q4 IRFS7530, Q5 IRFS7530, Q6 IRFS7530, U1 STM32F40X_LQFP64, U2 TC2117, U3 DRV8302, U401 SN65HVD232, X1 MINI-USB-SHIELD-32005-201, X2 8MHz 10ppm

Commit message: more changes
Parts:
- moved J4 2.75 mm to (73.3, 105.5)
- moved J5 1.50 mm to (73.5, 119.0)
Routing:
- net V_SUPPLY: vias 20 -> 32
- added copper zone on B.Cu, net V_SUPPLY
Other:
- board size 38.5 x 75 mm -> 48.5 x 75 mm
Changed lines of the file:
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@@
 	(footprint "vesc:7466103"
 		(layer "B.Cu")
-		(at 72 119 180)
+		(at 73.5 119 180)
 		(descr "7466103-3")
 		(tags "Connector")
 		(property "Reference" "J5"
-			(at 0 0 0)
+			(at -2 0 0)
 			(layer "B.SilkS")
 			(effects
@@
 	(footprint "vesc:7466103"
 		(layer "B.Cu")
-		(at 71 107 180)
+		(at 73.3 105.5 180)
 		(descr "7466103-3")
 		(tags "Connector")
@@
 		)
 	)
-	(gr_line
-		(start 74.93 131.826)
-		(end 74.93 123.825)
-		(stroke
-			(width 0.2)
-			(type solid)
-		)
-		(layer "Dwgs.User")
-	)
-	(gr_line
-		(start 74.93 123.825)
-		(end 78.486 123.825)
-		(stroke
-			(width 0.2)
-			(type solid)
-		)
-		(layer "Dwgs.User")
-	)
-	(gr_line
-		(start 78.486 131.826)
-		(end 74.93 131.826)
-		(stroke
-			(width 0.2)
-			(type solid)
-		)
-		(layer "Dwgs.User")
-	)
 	(gr_arc
 		(start 110 139)
@@
 	(gr_line
 		(start 84.5 145)
-		(end 78.5 145)
+		(end 68.5 145)
 		(stroke
 			(width 0.15)
@@
 	)
 	(gr_line
-		(start 78.5 145)
-		(end 78.5 70)
+		(start 68.5 145)
+		(end 68.5 70)
 		(stroke
 			(width 0.15)
@@
 	(gr_line
 		(start 117 70)
-		(end 78.5 70)
+		(end 68.5 70)
 		(stroke
 			(width 0.15)
@@
 	)
 	(segment
-		(start 81.788 100.76942)
-		(end 84.709 97.84842)
-		(width 5.08)
-		(layer "F.Cu")
-		(net 41)
-	)
-	(segment
 		(start 81.788 106.172)
 		(end 90.11158 97.84842)
@@
 	)
 	(segment
+		(start 81.788 108.966)
+		(end 81.788 100.76942)
+		(width 5.08)
+		(layer "F.Cu")
+		(net 41)
+	)
+	(segment
 		(start 97.917 97.84842)
 		(end 95.30842 97.84842)
@@
 	)
 	(segment
-		(start 81.788 108.966)
-		(end 81.788 100.76942)
-		(width 5.08)
-		(layer "F.Cu")
-		(net 41)
-	)
-	(segment
 		(start 96.65716 111.8235)
 		(end 96.4565 111.8235)
@@
 	)
 	(segment
+		(start 81.788 100.76942)
+		(end 84.709 97.84842)
+		(width 5.08)
+		(layer "F.Cu")
+		(net 41)
+	)
+	(segment
 		(start 112.20958 99.314)
 		(end 110.744 97.84842)
@@
 	)
 	(via
+		(at 74.2 98.2)
+		(size 1.524)
+		(drill 0.762)
+		(layers "F.Cu" "B.Cu")
+		(net 41)
+	)
+	(via
 		(at 116.078 99.314)
 		(size 0.8)
@@
 	)
 	(via
+		(at 69.4 98.2)
+		(size 1.524)
+		(drill 0.762)
+		(layers "F.Cu" "B.Cu")
+		(net 41)
+	)
+	(via
 		(at 80.01 110.744)
 		(size 1.524)
@@
 	)
 	(via
+		(at 75.8 99.9)
+		(size 1.524)
+		(drill 0.762)
+		(layers "F.Cu" "B.Cu")
+		(net 41)
+	)
+	(via
 		(at 80.01 107.188)
 		(size 1.524)
@@
 	)
 	(via
+		(at 75.8 98.2)
+		(size 1.524)
+		(drill 0.762)
+		(layers "F.Cu" "B.Cu")
+		(net 41)
+	)
+	(via
 		(at 83.566 108.966)
 		(size 1.524)
@@
 	)
 	(via
+		(at 77.4 98.2)
+		(size 1.524)
+		(drill 0.762)
+		(layers "F.Cu" "B.Cu")
+		(net 41)
+	)
+	(via
 		(at 81.788 108.966)
 		(size 1.524)
@@
 	)
 	(via
+		(at 77.4 99.9)
+		(size 1.524)
+		(drill 0.762)
+		(layers "F.Cu" "B.Cu")
+		(net 41)
+	)
+	(via
 		(at 80.01 108.966)
 		(size 1.524)
@@
 	)
 	(via
+		(at 72.6 98.2)
+		(size 1.524)
+		(drill 0.762)
+		(layers "F.Cu" "B.Cu")
+		(net 41)
+	)
+	(via
+		(at 69.4 99.9)
+		(size 1.524)
+		(drill 0.762)
+		(layers "F.Cu" "B.Cu")
+		(net 41)
+	)
+	(via
+		(at 71 99.9)
+		(size 1.524)
+		(drill 0.762)
+		(layers "F.Cu" "B.Cu")
+		(net 41)
+	)
+	(via
 		(at 96.647 114.046)
 		(size 0.8)
@@
 	)
 	(via
+		(at 74.2 99.9)
+		(size 1.524)
+		(drill 0.762)
+		(layers "F.Cu" "B.Cu")
+		(net 41)
+	)
+	(via
 		(at 83.566 107.188)
 		(size 1.524)
@@
 	)
 	(via
+		(at 72.6 99.9)
+		(size 1.524)
+		(drill 0.762)
+		(layers "F.Cu" "B.Cu")
+		(net 41)
+	)
+	(via
+		(at 71 98.2)
+		(size 1.524)
+		(drill 0.762)
+		(layers "F.Cu" "B.Cu")
+		(net 41)
+	)
+	(via
 		(at 81.788 110.744)
 		(size 1.524)
@@
 		(polygon
 			(pts
-				(xy 89.027 108.585) (xy 89.027 102.235) (xy 82.804 102.235) (xy 82.804 108.585)
+				(xy 89.027 108.585) (xy 89.027 102.235) (xy 78.2 102.3) (xy 78.2 97.3) (xy 68.504 97.3) (xy 68.504 108.685)
 			)
 		)
@@
 		(polygon
 			(pts
-				(xy 117 139) (xy 78.5 139) (xy 78.5 110) (xy 94.996 109.982) (xy 94.996 108.077) (xy 92.71 108.077)
-				(xy 92.71 97.155) (xy 100.838 97.155) (xy 100.838 102.997) (xy 101.727 102.997) (xy 101.727 108.077)
-				(xy 100.33 108.077) (xy 100.33 109.982) (xy 117 110)
+				(xy 117 139) (xy 78.5 139) (xy 78.5 133) (xy 68.5 133) (xy 68.5 114) (xy 78.5 114) (xy 78.5 110)
+				(xy 94.996 109.982) (xy 94.996 108.077) (xy 92.71 108.077) (xy 92.71 97.155) (xy 100.838 97.155)
+				(xy 100.838 102.997) (xy 101.727 102.997) (xy 101.727 108.077) (xy 100.33 108.077) (xy 100.33 109.982)
+				(xy 117 110)
 			)
 		)
@@
 			)
 		)
+	)
+	(zone
+		(net 41)
+		(net_name "V_SUPPLY")
+		(layer "B.Cu")
+		(hatch edge 0.5)
+		(priority 1)
+		(connect_pads
+			(clearance 0.508)
+		)
+		(min_thickness 0.25)
+		(filled_areas_thickness no)
+		(fill yes
+			(thermal_gap 0.5)
+			(thermal_bridge_width 0.5)
+		)
+		(polygon
+			(pts
+				(xy 68.5 97.3) (xy 68.5 112) (xy 78.2 111.9) (xy 78.2 97.3)
+			)
+		)

Commit message: changees
Other:
- board size 48.5 x 75 mm -> 48.4 x 75 mm
Changed lines of the file:
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@@
 		)
 		(sheetname "Root")
-		(sheetfile "C:/Electrical/bldc-hardware-master/design/BLDC_4.sch")
+		(sheetfile "BLDC_4.kicad_sch")
 		(attr through_hole)
 		(fp_line
@@
 		)
 		(sheetname "Root")
-		(sheetfile "C:/Electrical/bldc-hardware-master/design/BLDC_4.sch")
+		(sheetfile "BLDC_4.kicad_sch")
 		(attr through_hole)
 		(fp_line
@@
 		)
 		(sheetname "Root")
-		(sheetfile "C:/Electrical/bldc-hardware-master/design/BLDC_4.sch")
+		(sheetfile "BLDC_4.kicad_sch")
 		(attr through_hole)
 		(fp_line
@@
 		)
 		(sheetname "Root")
-		(sheetfile "C:/Electrical/bldc-hardware-master/design/BLDC_4.sch")
+		(sheetfile "BLDC_4.kicad_sch")
 		(attr through_hole)
 		(fp_line
@@
 		)
 		(sheetname "Root")
-		(sheetfile "C:/Electrical/bldc-hardware-master/design/BLDC_4.sch")
+		(sheetfile "BLDC_4.kicad_sch")
 		(attr through_hole)
 		(fp_line
@@
 		)
 		(sheetname "Root")
-		(sheetfile "C:/Electrical/bldc-hardware-master/design/BLDC_4.sch")
+		(sheetfile "BLDC_4.kicad_sch")
 		(attr through_hole)
 		(fp_line
@@
 		(property ki_fp_filters "R? SM0603 SM0805 R?-* SM1206")
 		(sheetname "Root")
-		(sheetfile "C:/Electrical/bldc-hardware-master/design/BLDC_4.sch")
+		(sheetfile "BLDC_4.kicad_sch")
 		(attr smd)
 		(fp_line
@@
 		(property ki_fp_filters "R? SM0603 SM0805 R?-* SM1206")
 		(sheetname "Root")
-		(sheetfile "C:/Electrical/bldc-hardware-master/design/BLDC_4.sch")
+		(sheetfile "BLDC_4.kicad_sch")
 		(attr smd)
 		(fp_line
@@
 		)
 		(sheetname "Root")
-		(sheetfile "C:/Electrical/bldc-hardware-master/design/BLDC_4.sch")
+		(sheetfile "BLDC_4.kicad_sch")
 		(attr smd)
 		(fp_line
@@
 		(property ki_fp_filters "Pin_Header_Straight_1X07 Pin_Header_Angled_1X07 Socket_Strip_Straight_1X07 Socket_Strip_Angled_1X07")
 		(sheetname "Root")
-		(sheetfile "C:/Electrical/bldc-hardware-master/design/BLDC_4.sch")
+		(sheetfile "BLDC_4.kicad_sch")
 		(attr through_hole)
 		(fp_line
@@
 		(property ki_fp_filters "LED-3MM LED-5MM LED-10MM LED-0603 LED-0805 LED-1206 LEDV")
 		(sheetname "Root")
-		(sheetfile "C:/Electrical/bldc-hardware-master/design/BLDC_4.sch")
+		(sheetfile "BLDC_4.kicad_sch")
 		(attr smd)
 		(fp_line
@@
 		(property ki_fp_filters "LED-3MM LED-5MM LED-10MM LED-0603 LED-0805 LED-1206 LEDV")
 		(sheetname "Root")
-		(sheetfile "C:/Electrical/bldc-hardware-master/design/BLDC_4.sch")
+		(sheetfile "BLDC_4.kicad_sch")
 		(attr smd)
 		(fp_line
@@
 		(property ki_fp_filters "LED-3MM LED-5MM LED-10MM LED-0603 LED-0805 LED-1206 LEDV")
 		(sheetname "Root")
-		(sheetfile "C:/Electrical/bldc-hardware-master/design/BLDC_4.sch")
+		(sheetfile "BLDC_4.kicad_sch")
 		(attr smd)
 		(fp_line
@@
 		)
 		(sheetname "Root")
-		(sheetfile "C:/Electrical/bldc-hardware-master/design/BLDC_4.sch")
+		(sheetfile "BLDC_4.kicad_sch")
 		(attr through_hole)
 		(fp_line
@@
 		)
 		(sheetname "Root")
-		(sheetfile "C:/Electrical/bldc-hardware-master/design/BLDC_4.sch")
+		(sheetfile "BLDC_4.kicad_sch")
 		(attr through_hole)
 		(fp_line
@@
 		(property ki_fp_filters "R? SM0603 SM0805 R?-* SM1206")
 		(sheetname "Root")
-		(sheetfile "C:/Electrical/bldc-hardware-master/design/BLDC_4.sch")
+		(sheetfile "BLDC_4.kicad_sch")
 		(attr smd)
 		(fp_line
@@
 		(property ki_fp_filters "R? SM0603 SM0805 R?-* SM1206")
 		(sheetname "Root")
-		(sheetfile "C:/Electrical/bldc-hardware-master/design/BLDC_4.sch")
+		(sheetfile "BLDC_4.kicad_sch")
 		(attr smd)
 		(fp_line
@@
 		(property ki_fp_filters "SM* C? C1-1")
 		(sheetname "Root")
-		(sheetfile "C:/Electrical/bldc-hardware-master/design/BLDC_4.sch")
+		(sheetfile "BLDC_4.kicad_sch")
 		(attr smd)
 		(fp_line
@@
 		(property ki_fp_filters "SM* C? C1-1")
 		(sheetname "Root")
-		(sheetfile "C:/Electrical/bldc-hardware-master/design/BLDC_4.sch")
+		(sheetfile "BLDC_4.kicad_sch")
 		(attr smd)
 		(fp_line
@@
 		(property ki_fp_filters "R? SM0603 SM0805 R?-* SM1206")
 		(sheetname "Root")
-		(sheetfile "C:/Electrical/bldc-hardware-master/design/BLDC_4.sch")
+		(sheetfile "BLDC_4.kicad_sch")
 		(attr smd)
 		(fp_line
@@
 		(property ki_fp_filters "R? SM0603 SM0805 R?-* SM1206")
 		(sheetname "Root")
-		(sheetfile "C:/Electrical/bldc-hardware-master/design/BLDC_4.sch")
+		(sheetfile "BLDC_4.kicad_sch")
 		(attr smd)
 		(fp_line
@@
 		(property ki_fp_filters "R? SM0603 SM0805 R?-* SM1206")
 		(sheetname "Root")
-		(sheetfile "C:/Electrical/bldc-hardware-master/design/BLDC_4.sch")
+		(sheetfile "BLDC_4.kicad_sch")
 		(attr smd)
 		(fp_line
@@
 		(property ki_fp_filters "R? SM0603 SM0805 R?-* SM1206")
 		(sheetname "Root")
-		(sheetfile "C:/Electrical/bldc-hardware-master/design/BLDC_4.sch")
+		(sheetfile "BLDC_4.kicad_sch")
 		(attr smd)
 		(fp_line
@@
 		(property ki_fp_filters "R? SM0603 SM0805 R?-* SM1206")
 		(sheetname "Root")
-		(sheetfile "C:/Electrical/bldc-hardware-master/design/BLDC_4.sch")
+		(sheetfile "BLDC_4.kicad_sch")
 		(attr smd)
 		(fp_line
@@
 		(property ki_fp_filters "R? SM0603 SM0805 R?-* SM1206")
 		(sheetname "Root")
-		(sheetfile "C:/Electrical/bldc-hardware-master/design/BLDC_4.sch")
+		(sheetfile "BLDC_4.kicad_sch")
 		(attr smd)
 		(fp_line
@@
 		(property ki_fp_filters "R? SM0603 SM0805 R?-* SM1206")
 		(sheetname "Root")
-		(sheetfile "C:/Electrical/bldc-hardware-master/design/BLDC_4.sch")
+		(sheetfile "BLDC_4.kicad_sch")
 		(attr smd)
 		(fp_line
@@
 		)
 		(property "Height" "7"
-			(at 0 0 0)
+			(at 0 0 180)
 			(unlocked yes)
 			(layer "B.Fab")
@@
 		)
 		(property "Manufacturer_Name" "Wurth Elektronik"
-			(at 0 0 0)
+			(at 0 0 180)
 			(unlocked yes)
 			(layer "B.Fab")
@@
 		)
 		(property "Manufacturer_Part_Number" "7466103"
-			(at 0 0 0)
+			(at 0 0 180)
 			(unlocked yes)
 			(layer "B.Fab")
@@
 		)
 		(property "Arrow Part Number" ""
-			(at 0 0 0)
+			(at 0 0 180)
 			(unlocked yes)
 			(layer "B.Fab")
@@
 		)
 		(property "Arrow Price/Stock" ""
-			(at 0 0 0)
+			(at 0 0 180)
 			(unlocked yes)
 			(layer "B.Fab")
@@
 		)
 		(property "Height" "7"
-			(at 0 0 0)
+			(at 0 0 180)
 			(unlocked yes)
 			(layer "B.Fab")
@@
 		)
 		(property "Manufacturer_Name" "Wurth Elektronik"
-			(at 0 0 0)
+			(at 0 0 180)
 			(unlocked yes)
 			(layer "B.Fab")
@@
 		)
 		(property "Manufacturer_Part_Number" "7466103"
-			(at 0 0 0)
+			(at 0 0 180)
 			(unlocked yes)
 			(layer "B.Fab")
@@
 		)
 		(property "Arrow Part Number" ""
-			(at 0 0 0)
+			(at 0 0 180)
 			(unlocked yes)
 			(layer "B.Fab")
@@
 		)
 		(property "Arrow Price/Stock" ""
-			(at 0 0 0)
+			(at 0 0 180)
 			(unlocked yes)
 			(layer "B.Fab")
@@
 		(tags "Connector")
 		(property "Reference" "J5"
-			(at -2 0 0)
+			(at 0 0 0)
 			(layer "B.SilkS")
 			(effects
@@
 		)
 		(property "Height" "7"
-			(at 0 0 0)
+			(at 0 0 180)
 			(unlocked yes)
 			(layer "B.Fab")
@@
 		)
 		(property "Manufacturer_Name" "Wurth Elektronik"
-			(at 0 0 0)
+			(at 0 0 180)
 			(unlocked yes)
 			(layer "B.Fab")
@@
 		)
 		(property "Manufacturer_Part_Number" "7466103"
-			(at 0 0 0)
+			(at 0 0 180)
 			(unlocked yes)
 			(layer "B.Fab")
@@
 		)
 		(property "Arrow Part Number" ""
-			(at 0 0 0)
+			(at 0 0 180)
 			(unlocked yes)
 			(layer "B.Fab")
@@
 		)
 		(property "Arrow Price/Stock" ""
-			(at 0 0 0)
+			(at 0 0 180)
 			(unlocked yes)
 			(layer "B.Fab")
@@
 		)
 		(property "Height" "7"
-			(at 0 0 0)
+			(at 0 0 180)
 			(unlocked yes)
 			(layer "B.Fab")
@@
 		)
 		(property "Manufacturer_Name" "Wurth Elektronik"
-			(at 0 0 0)
+			(at 0 0 180)
 			(unlocked yes)
 			(layer "B.Fab")
@@
 		)
 		(property "Manufacturer_Part_Number" "7466103"
-			(at 0 0 0)
+			(at 0 0 180)
 			(unlocked yes)
 			(layer "B.Fab")
@@
 		)
 		(property "Arrow Part Number" ""
-			(at 0 0 0)
+			(at 0 0 180)
 			(unlocked yes)
 			(layer "B.Fab")
@@
 		)
 		(property "Arrow Price/Stock" ""
-			(at 0 0 0)
+			(at 0 0 180)
 			(unlocked yes)
 			(layer "B.Fab")
@@
 		)
 		(property "Height" "7"
-			(at 0 0 0)
+			(at 0 0 180)
 			(unlocked yes)
 			(layer "B.Fab")
@@
 		)
 		(property "Manufacturer_Name" "Wurth Elektronik"
-			(at 0 0 0)
+			(at 0 0 180)
 			(unlocked yes)
 			(layer "B.Fab")
@@
 		)
 		(property "Manufacturer_Part_Number" "7466103"
-			(at 0 0 0)
+			(at 0 0 180)
 			(unlocked yes)
 			(layer "B.Fab")
@@
 		)
 		(property "Arrow Part Number" ""
-			(at 0 0 0)
+			(at 0 0 180)
 			(unlocked yes)
 			(layer "B.Fab")
@@
 		)
 		(property "Arrow Price/Stock" ""
-			(at 0 0 0)
+			(at 0 0 180)
 			(unlocked yes)
 			(layer "B.Fab")
@@
 	(gr_line
 		(start 84.5 145)
-		(end 68.5 145)
+		(end 78.6 145)
 		(stroke
 			(width 0.15)
@@
 	)
 	(gr_line
-		(start 68.5 145)
-		(end 68.5 70)
+		(start 68.617503 135.100344)
+		(end 68.6 79.9)
 		(stroke
 			(width 0.15)
@@
 	(gr_line
 		(start 117 70)
-		(end 68.5 70)
+		(end 78.5 70)
 		(stroke
 			(width 0.15)
@@
 		)
 		(layer "Edge.Cuts")
+	)
+	(gr_arc
+		(start 78.6 145)
+		(mid 71.546374 142.129808)
+		(end 68.617503 135.100344)
+		(stroke
+			(width 0.15)
+			(type default)
+		)
+		(layer "Edge.Cuts")
+	)
+	(gr_arc
+		(start 68.6 79.9)
+		(mid 71.499643 72.899643)
+		(end 78.5 70)
+		(stroke
+			(width 0.15)
+			(type default)
+		)
+		(layer "Edge.Cuts")

Commit message: changes
Parts:
- moved J5 0.20 mm to (73.3, 119.0)
Changed lines of the file:
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@@
 	(footprint "vesc:7466103"
 		(layer "B.Cu")
-		(at 73.5 119 180)
+		(at 73.3 119 180)
 		(descr "7466103-3")
 		(tags "Connector")
