File: bldc-hardware-master/design/BLDC_4.kicad_pcb (KiCad board)
At the start: 4 copper layers, 48.4 x 75 mm, 132 parts, among them J1 7466103, J2 7466103, J3 7466103, J4 7466103, J5 7466103, K1 SERVO, P1 HALL/Encoder, P101 CANBUS, P2 SWD, P3 PWR_COMM, P4 IN+, P5 IN-, P6 MOTOR1, P7 MOTOR2, P9 MOTOR3, Q1 IRFS7530, Q2 IRFS7530, Q3 IRFS7530, Q4 IRFS7530, Q5 IRFS7530, Q6 IRFS7530, U1 STM32F40X_LQFP64, U2 TC2117, U3 DRV8302, U401 SN65HVD232, X1 MINI-USB-SHIELD-32005-201, X2 8MHz 10ppm

Commit message: small changes
Other:
- board size 48.4 x 75 mm -> 48.5 x 75 mm
Changed lines of the file:
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@@
 	(gr_line
 		(start 84.5 145)
-		(end 78.6 145)
+		(end 78.5 145)
 		(stroke
 			(width 0.15)
@@
 	)
 	(gr_line
-		(start 68.617503 135.100344)
-		(end 68.6 79.9)
+		(start 68.5 123.528916)
+		(end 68.484857 96.583566)
 		(stroke
 			(width 0.15)
@@
 		(layer "Edge.Cuts")
 	)
-	(gr_arc
-		(start 78.6 145)
-		(mid 71.546374 142.129808)
-		(end 68.617503 135.100344)
+	(gr_line
+		(start 78.5 145)
+		(end 78.499999 133.470492)
 		(stroke
 			(width 0.15)
@@
 	)
 	(gr_arc
-		(start 68.6 79.9)
-		(mid 71.499643 72.899643)
-		(end 78.5 70)
+		(start 68.5 123.528874)
+		(mid 75.558883 126.428709)
+		(end 78.499998 133.470492)
 		(stroke
 			(width 0.15)
+			(type default)
+		)
+		(layer "Edge.Cuts")
+	)
+	(gr_line
+		(start 78.5 70)
+		(end 78.5 88)
+		(stroke
+			(width 0.15)
+			(type default)
+		)
+		(layer "Edge.Cuts")
+	)
+	(gr_arc
+		(start 78.499999 88)
+		(mid 74.991856 94.041287)
+		(end 68.484857 96.583566)
+		(stroke
+			(width 0.15)
